Commit message: Robot description: load fixed sensor mounting transforms from YAML in Xacro

File: ros/src/leroy_description/urdf/leroy.urdf.xacro (robot description, xacro)
@@ -3,20 +3,30 @@
   <!-- Body frames: +x forward, +y left, +z up -->
   <!-- Optical frames: +x right, +y down, +z forward -->
+  <!-- All hardware-specific fixed sensor mounting coordinates are in YAML.
+       The optical-axis conversion joints below are ROS frame conventions. -->
+  <xacro:arg name="sensor_mounts_file"
+             default="$(find leroy_description)/config/sensor_mounts.yaml"/>
+  <xacro:property name="mount_config"
+                  value="${xacro.load_yaml('$(arg sensor_mounts_file)')}"/>
+  <xacro:property name="mounts" value="${mount_config['mounts']}"/>
+  <xacro:macro name="sensor_origin" params="sensor">
+    <origin xyz="${mounts[sensor]['xyz'][0]} ${mounts[sensor]['xyz'][1]} ${mounts[sensor]['xyz'][2]}"
+            rpy="${mounts[sensor]['rpy'][0]} ${mounts[sensor]['rpy'][1]} ${mounts[sensor]['rpy'][2]}"/>
+  </xacro:macro>
   <link name="base_link"/>
-  <!-- PROVISIONAL: 95 mm forward, 95 mm right; IMU height and alignment
-       must be measured/verified before XRSLAM pose output is enabled. -->
+  <!-- PROVISIONAL IMU sensor centre, configured in sensor_mounts.yaml;
+       the MCU output is ALREADY robot-aligned. -->
   <link name="imu_link"/>
   <joint name="base_to_imu" type="fixed">
     <parent link="base_link"/>
     <child link="imu_link"/>
-    <origin xyz="0.095 -0.095 0.0" rpy="0 0 0"/>
+    <xacro:sensor_origin sensor="imu"/>
   </joint>
-  <!-- PROVISIONAL: front camera 30 deg below forward, zero translation.
-       Replace xyz/rpy with measured extrinsics in this canonical Xacro. -->
+  <!-- PROVISIONAL front camera mounting transform from YAML. -->
   <link name="front_camera_link"/>
   <joint name="base_to_front_camera" type="fixed">
     <parent link="base_link"/>
     <child link="front_camera_link"/>
-    <origin xyz="0 0 0" rpy="0 0.5235987755982988 0"/>
+    <xacro:sensor_origin sensor="front_camera"/>
   </joint>
   <link name="front_camera_optical_frame"/>
@@ -37,11 +47,10 @@
     <origin xyz="0 0 0" rpy="0 0 0"/>
   </joint>
-  <!-- PROVISIONAL: workspace camera 60 deg below forward, zero translation.
-       Replace xyz/rpy only after measurement. -->
+  <!-- PROVISIONAL workspace camera mounting transform from YAML. -->
   <link name="workspace_camera_link"/>
   <joint name="base_to_workspace_camera" type="fixed">
     <parent link="base_link"/>
     <child link="workspace_camera_link"/>
-    <origin xyz="0 0 0" rpy="0 1.0471975511965976 0"/>
+    <xacro:sensor_origin sensor="workspace_camera"/>
   </joint>
   <link name="workspace_camera_optical_frame"/>

Commit message: Robot description: explicitly resolve Xacro YAML argument before loading mounts

File: ros/src/leroy_description/urdf/leroy.urdf.xacro (robot description, xacro)
@@ -7,6 +7,7 @@
   <xacro:arg name="sensor_mounts_file"
              default="$(find leroy_description)/config/sensor_mounts.yaml"/>
+  <xacro:property name="mount_file_path" value="$(arg sensor_mounts_file)"/>
   <xacro:property name="mount_config"
-                  value="${xacro.load_yaml('$(arg sensor_mounts_file)')}"/>
+                  value="${xacro.load_yaml(mount_file_path)}"/>
   <xacro:property name="mounts" value="${mount_config['mounts']}"/>
   <xacro:macro name="sensor_origin" params="sensor">
